Commit message: urdf -> wrong mesh pose

File: urdf/pirov.xacro (robot description, xacro)
@@ -85,5 +85,5 @@
   <link name="base_link">
     <visual>
-      <origin xyz="-0.241 0.165 0.17" rpy="${-PI/2} 0 -${PI/2}"/>
+      <origin xyz="-0.241 0.165 0.17" rpy="${PI/2} 0 -${PI/2}"/>
       <!--origin xyz="-0.241 0.165 0.17" rpy="${PI/2} 0 -${PI/2}"/-->
       <geometry>
@@ -92,5 +92,5 @@
     </visual>
      <inertial>
-      <origin xyz="0 0 0.1" rpy="0 0 0"/>
+      <origin xyz="0 0 -0.1" rpy="0 0 0"/>
       <mass value="5"/>
       <inertia
@@ -105,9 +105,28 @@
       <compensation>1.01</compensation>
       <origin xyz= "0 0 0"/>
-      <limit radius=".1"/>
+      <limit radius="0.05"/>
       <damping xyz="50 100 60" rpy="50 50 50"/>
   </buoyancy>
   </link>
-  <link name="camera"/>
+  <link name="camera">
+    <visual>
+      <geometry>
+        <cylinder radius="0.01" length="0.03"/>
+      </geometry>
+    </visual>
+     <inertial>
+      <mass value="0.001"/>
+      <inertia
+	  ixx="0.001"
+	  ixy="0.0"
+	  ixz="0.0"
+	  iyy="0.001"
+	  iyz="0"
+	  izz="0.001"/>
+    </inertial>
+  </link>
+    <gazebo reference="camera">
+        <material>Gazebo/Black</material>
+    </gazebo>
   <joint name="tilt" type="revolute">
     <parent link="base_link"/>

Commit message: better thruster calibration

File: urdf/pirov.xacro (robot description, xacro)
@@ -4,10 +4,12 @@
   <xacro:property name="PI" value="3.1415926535897931"/>
   <!-- Body properties -->
-  <xacro:property name="thr12_y" value="0.115"/>
-  <xacro:property name="thr34_x" value="0.18"/>
-  <xacro:property name="thr34_y" value="0.1092"/>
-  <xacro:property name="thr5_x" value="0.17"/>
-  <xacro:property name="thr6_x" value="0.039"/>
-  <xacro:property name="thr56_z" value="0.105"/>
+  <xacro:property name="thr12_y" value="0.109"/>
+  <xacro:property name="thr1234_z" value="-0.02"/>
+  <xacro:property name="thr34_x" value="0.165"/>
+  <xacro:property name="thr34_y" value="0.11"/>
+  <xacro:property name="thr5_x" value="-0.185"/>
+  <xacro:property name="thr5_z" value="-0.105"/>
+  <xacro:property name="thr6_x" value="0.028"/>
+  <xacro:property name="thr6_z" value="-0.127"/>
   <xacro:property name="eps" value="0.00000001"/>
   <!-- Thruster link -->
@@ -54,30 +56,30 @@
             <effort>40</effort>
             <name>thr1</name>
-            <map>1 0 0 0 0 ${-thr12_y}</map>
+            <map>1 0 0 0 0 ${thr12_y}</map>
         </thruster>
         <thruster>
             <effort>40</effort>
             <name>thr2</name>
-            <map>1 0 0 0 0 ${thr12_y}</map>
+            <map>1 0 0 0 0 ${-thr12_y}</map>
         </thruster>
         <thruster>
             <effort>30</effort>
             <name>thr3</name>
+            <map>0 0 -1 ${thr34_y} ${thr34_x} 0</map>
+        </thruster>
+        <thruster>
+            <effort>30</effort>
+            <name>thr4</name>
             <map>0 0 -1 ${-thr34_y} ${thr34_x} 0</map>
         </thruster>
         <thruster>
             <effort>30</effort>
-            <name>thr4</name>
-            <map>0 0 -1 ${thr34_y} ${thr34_x} 0</map>
-        </thruster>
-        <thruster>
-            <effort>30</effort>
             <name>thr5</name>
-            <map>0 0 -1 0 ${-thr5_x} 0</map>
+            <map>0 0 -1 0 ${thr5_x} 0</map>
         </thruster>
         <thruster>
             <effort>30</effort>
             <name>thr6</name>
-            <map>0 1 0 ${-thr56_z} 0 0</map>
+            <map>0 1 0 ${-thr6_z} 0 0</map>
         </thruster>
     </plugin>
@@ -85,5 +87,5 @@
   <link name="base_link">
     <visual>
-      <origin xyz="-0.241 0.165 0.17" rpy="${PI/2} 0 -${PI/2}"/>
+      <origin xyz="-0.253 -0.167 -0.19" rpy="${PI/2} 0 ${PI/2}"/>
       <!--origin xyz="-0.241 0.165 0.17" rpy="${PI/2} 0 -${PI/2}"/-->
       <geometry>
@@ -109,4 +111,10 @@
   </buoyancy>
   </link>
+  <link name="body"/>
+  <joint name="body_offset" type="fixed">
+    <parent link="base_link"/>
+    <child link="body"/>
+    <origin xyz="0.02 0 0"/>
+  </joint>
   <link name="camera">
     <visual>
@@ -125,4 +133,5 @@
 	  izz="0.001"/>
     </inertial>
+    <origin rpy="0 {PI/2} 0"/>
   </link>
     <gazebo reference="camera">
@@ -130,7 +139,8 @@
     </gazebo>
   <joint name="tilt" type="revolute">
-    <parent link="base_link"/>
+    <parent link="body"/>
     <child link="camera"/>
-    <origin rpy="${PI/2} 0 0" xyz="0.15 0 0"/>
+    <origin xyz="0.15 0 0"/>
+    <axis xyz="0 1 0" />
     <limit effort="100" velocity="5.0" lower="${-PI/4}" upper="${PI/4}"/>
   </joint>
@@ -138,12 +148,12 @@
   <link name="mpu"/>
   <joint name="lsm" type="fixed">
-    <parent link="base_link"/>
+    <parent link="body"/>
     <child link="lsm"/>
-    <origin rpy="0 0 0" xyz="0.1 0.018 0.05"/>
+    <origin rpy="0 0 0" xyz="0.1 0.018 0.02"/>
   </joint>
     <joint name="mpu" type="fixed">
-    <parent link="base_link"/>
+    <parent link="body"/>
     <child link="mpu"/>
-    <origin rpy="0 0 0" xyz="0.11 0.018 0.05"/>
+    <origin rpy="0 0 0" xyz="0.11 0.018 0.02"/>
   </joint>
     <gazebo reference="lsm">
@@ -183,9 +193,9 @@
     </sensor>
    </gazebo>
-<xacro:thruster_dummy_link name="thr1" xyz="0.0 0.115 0.0" rpy="-0.0 -1.57079632679 0.0"/>
-<xacro:thruster_dummy_link name="thr2" xyz="0.0 -0.115 0.0" rpy="-0.0 -1.57079632679 0.0"/>
-<xacro:thruster_dummy_link name="thr3" xyz="0.18 0.1092 0.0" rpy="0.0 -0.0 0.0"/>
-<xacro:thruster_dummy_link name="thr4" xyz="0.18 -0.1092 0.0" rpy="0.0 -0.0 0.0"/>
-<xacro:thruster_dummy_link name="thr5" xyz="-0.17 0.0 0.0" rpy="0.0 -0.0 0.0"/>
-<xacro:thruster_dummy_link name="thr6" xyz="0.0 0.0 0.105" rpy="1.57079632679 -0.0 0.0"/>
+<xacro:thruster_dummy_link name="thr1" xyz="0.0 ${-thr12_y} ${thr1234_z}" rpy="-0.0 -1.57079632679 0.0"/>
+<xacro:thruster_dummy_link name="thr2" xyz="0.0 ${thr12_y} ${thr1234_z}" rpy="-0.0 -1.57079632679 0.0"/>
+<xacro:thruster_dummy_link name="thr3" xyz="${thr34_x} ${-thr34_y} ${thr1234_z}" rpy="0.0 -0.0 0.0"/>
+<xacro:thruster_dummy_link name="thr4" xyz="${thr34_x} ${thr34_y} ${thr1234_z}" rpy="0.0 -0.0 0.0"/>
+<xacro:thruster_dummy_link name="thr5" xyz="${thr5_x} 0.0 ${thr5_z}" rpy="0.0 -0.0 0.0"/>
+<xacro:thruster_dummy_link name="thr6" xyz="${thr6_x} 0.0 ${thr6_z}" rpy="1.57079632679 -0.0 0.0"/>
 </robot>

Commit message: RViz displays only rotation

File: urdf/pirov.xacro (robot description, xacro)
@@ -119,4 +119,5 @@
   <link name="camera">
     <visual>
+        <origin rpy="0 ${PI/2} 0"/>
       <geometry>
         <cylinder radius="0.01" length="0.03"/>
@@ -133,5 +134,4 @@
 	  izz="0.001"/>
     </inertial>
-    <origin rpy="0 {PI/2} 0"/>
   </link>
     <gazebo reference="camera">

Commit message: change Navio2 submobule

File: urdf/pirov.xacro (robot description, xacro)
@@ -111,5 +111,17 @@
   </buoyancy>
   </link>
-  <link name="body"/>
+  <link name="body">
+      <inertial>
+      <origin xyz="0 0 0" rpy="0 0 0"/>
+      <mass value="0.001"/>
+      <inertia
+	  ixx="0.001"
+	  ixy="0.0"
+	  ixz="0.0"
+	  iyy="0.001"
+	  iyz="0.001"
+	  izz="0.001"/>
+    </inertial>
+  </link>
   <joint name="body_offset" type="fixed">
     <parent link="base_link"/>
@@ -118,6 +130,6 @@
   </joint>
   <link name="camera">
+    <origin rpy="0 ${PI/2} 0"/>
     <visual>
-        <origin rpy="0 ${PI/2} 0"/>
       <geometry>
         <cylinder radius="0.01" length="0.03"/>

Commit message: tilt damping for simulation

File: urdf/pirov.xacro (robot description, xacro)
@@ -12,4 +12,5 @@
   <xacro:property name="thr6_x" value="0.028"/>
   <xacro:property name="thr6_z" value="-0.127"/>
+  <xacro:property name="x_offset" value="0.02"/>
   <xacro:property name="eps" value="0.00000001"/>
   <!-- Thruster link -->
@@ -107,32 +108,16 @@
       <compensation>1.01</compensation>
       <origin xyz= "0 0 0"/>
-      <limit radius="0.05"/>
+      <limit radius="0.01"/>
       <damping xyz="50 100 60" rpy="50 50 50"/>
   </buoyancy>
   </link>
-  <link name="body">
-      <inertial>
-      <origin xyz="0 0 0" rpy="0 0 0"/>
-      <mass value="0.001"/>
-      <inertia
-	  ixx="0.001"
-	  ixy="0.0"
-	  ixz="0.0"
-	  iyy="0.001"
-	  iyz="0.001"
-	  izz="0.001"/>
-    </inertial>
-  </link>
-  <joint name="body_offset" type="fixed">
-    <parent link="base_link"/>
-    <child link="body"/>
-    <origin xyz="0.02 0 0"/>
-  </joint>
   <link name="camera">
-    <origin rpy="0 ${PI/2} 0"/>
     <visual>
       <geometry>
         <cylinder radius="0.01" length="0.03"/>
       </geometry>
+      <material name="black">
+        <color rgba="0 0 0 1"/>
+    </material>
     </visual>
      <inertial>
@@ -151,21 +136,22 @@
     </gazebo>
   <joint name="tilt" type="revolute">
-    <parent link="body"/>
+    <parent link="base_link"/>
     <child link="camera"/>
-    <origin xyz="0.15 0 0"/>
+    <origin xyz="${x_offset + .15} 0 0" rpy="0 ${PI/2} 0"/>
     <axis xyz="0 1 0" />
     <limit effort="100" velocity="5.0" lower="${-PI/4}" upper="${PI/4}"/>
+    <dynamics damping="0.8"/>
   </joint>
   <link name="lsm"/>
   <link name="mpu"/>
   <joint name="lsm" type="fixed">
-    <parent link="body"/>
+    <parent link="base_link"/>
     <child link="lsm"/>
-    <origin rpy="0 0 0" xyz="0.1 0.018 0.02"/>
+    <origin rpy="0 0 0" xyz="${x_offset + .1} 0.018 0.02"/>
   </joint>
     <joint name="mpu" type="fixed">
-    <parent link="body"/>
+    <parent link="base_link"/>
     <child link="mpu"/>
-    <origin rpy="0 0 0" xyz="0.11 0.018 0.02"/>
+    <origin rpy="0 0 0" xyz="${x_offset + .11} 0.018 0.02"/>
   </joint>
     <gazebo reference="lsm">
@@ -174,8 +160,7 @@
       <update_rate>100</update_rate>
       <visualize>true</visualize>
-      <topic>lsm</topic>
       <plugin filename="libgazebo_ros_imu_sensor.so" name="imu_plugin">
         <topicName>lsm</topicName>
-        <bodyName>lsm</bodyName>
+        <bodyName>pirov</bodyName>
         <updateRateHZ>100.0</updateRateHZ>
         <gaussianNoise>0.01</gaussianNoise>
@@ -184,5 +169,4 @@
         <frameName>lsm</frameName>
       </plugin>
-      <pose>0 0 0 0 0 0</pose>
     </sensor>
    </gazebo>
@@ -192,8 +176,7 @@
       <update_rate>100</update_rate>
       <visualize>true</visualize>
-      <topic>mpu</topic>
       <plugin filename="libgazebo_ros_imu_sensor.so" name="imu_plugin">
         <topicName>mpu</topicName>
-        <bodyName>mpu</bodyName>
+        <bodyName>pirov</bodyName>
         <updateRateHZ>100.0</updateRateHZ>
         <gaussianNoise>0.01</gaussianNoise>
@@ -202,5 +185,4 @@
         <frameName>mpu</frameName>
       </plugin>
-      <pose>0 0 0 0 0 0</pose>
     </sensor>
    </gazebo>

File: urdf/pirov_uwsim.urdf (robot description, URDF)
Before this commit: robot pirov, 11 links, 10 joints
Links:
- link base_link: mass None -> 5; geometry visual mesh filename=file:///home/olivier/code/ros/src/bluerov/bluerov_ffg/mesh/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 scale=0.001 0.001 0.001
- link body: mass None -> 0.001
- link camera: mass None -> 0.001
Joints:
- joint tilt: origin xyz=0.15 0 0 -> xyz=0.15 0 0 rpy=0 1.57079632679 0

Commit message: only compile navio stuff on ROV

File: urdf/pirov.xacro (robot description, xacro)
@@ -91,5 +91,5 @@
       <!--origin xyz="-0.241 0.165 0.17" rpy="${PI/2} 0 -${PI/2}"/-->
       <geometry>
-	<mesh filename="file://$(find bluerov_ffg)/mesh/brov-redux.stl" scale="0.001 0.001 0.001"/>
+	<mesh filename="file://$(find ecn_bluerov_base)/mesh/brov-redux.stl" scale="0.001 0.001 0.001"/>
       </geometry>
     </visual>
